File: DC.kicad_pcb (KiCad board)
At the start: 4 copper layers, 199.5 x 140 mm, 107 parts, among them J1 348302001, J2 348302001, J3 757570141, J4 PPTC021LFBN-RC, Q1 BSS806NE, Q2 BSS806NE, Q3 BSS806NE, Q4 BSS806NE, Q5 BSS806NE, U1 MCP2551-I-P, U2 100DP6T1B1M1QEH, U5 NUCLEO-F302R8, U6 C1F 3

Commit message: gl lucas
Other:
- board text added: "8:AccelIn 7:BrakePedalIn 6:ThermalShutoff"
- board text added: "BLEDs 6-10"
- board text added: "CM"
- board text added: "EN"
- board text added: "FAULT"
- board text added: "FPChrg"
- board text added: "GLEDs 9,10 18-20"
- board text added: "HV"
- board text added: "HV+"
- board text added: "HV-"
- board text added: "HVIL"
- board text added: "Indicator LEDs 17-20"
- board text added: "LV"
- board text added: "LV+"
- board text added: "LV-"
- board text added: "Lights 1-6 11-16"
- board text added: "MS"
- board text added: "RM"
Changed lines of the file:
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@@
 			(plot_on_all_layers_selection 0x00000000_00000000_00000000_00000000)
 			(disableapertmacros no)
-			(usegerberextensions no)
-			(usegerberattributes yes)
-			(usegerberadvancedattributes yes)
+			(usegerberextensions yes)
+			(usegerberattributes no)
+			(usegerberadvancedattributes no)
 			(creategerberjobfile no)
 			(dashed_line_dash_ratio 12.000000)
@@
 			(plotpadnumbers no)
 			(hidednponfab no)
-			(sketchdnponfab yes)
-			(crossoutdnponfab yes)
+			(sketchdnponfab no)
+			(crossoutdnponfab no)
 			(subtractmaskfromsilk yes)
 			(outputformat 1)
@@
 			(at 1.675 -1.635 0)
 			(layer "F.SilkS")
+			(hide yes)
 			(effects
 				(font
@@
 		)
 	)
+	(gr_text "RM"
+		(at 113 196 0)
+		(layer "F.SilkS")
+		(effects
+			(font
+				(size 1.25 1.25)
+				(thickness 0.2)
+			)
+			(justify left bottom)
+		)
+	)
 	(gr_text "+12V"
 		(at 255 152.5 0)
@@
 		)
 	)
+	(gr_text "BLEDs \n6-10"
+		(at 85.5 192 0)
+		(layer "F.SilkS")
+		(effects
+			(font
+				(size 1.25 1.25)
+				(thickness 0.2)
+			)
+			(justify left bottom)
+		)
+	)
+	(gr_text "HV+"
+		(at 131 187 0)
+		(layer "F.SilkS")
+		(effects
+			(font
+				(size 1.25 1.25)
+				(thickness 0.2)
+			)
+			(justify left bottom)
+		)
+	)
 	(gr_text "+3V3\n"
 		(at 251 157 0)
@@
 		)
 	)
+	(gr_text "Lights\n1-6\n11-16"
+		(at 222 193.5 0)
+		(layer "F.SilkS")
+		(effects
+			(font
+				(size 1.25 1.25)
+				(thickness 0.2)
+			)
+			(justify left bottom)
+		)
+	)
 	(gr_text "Blue LEDs"
 		(at 123 159.5 0)
@@
 		)
 	)
+	(gr_text "EN"
+		(at 127 196 0)
+		(layer "F.SilkS")
+		(effects
+			(font
+				(size 1.25 1.25)
+				(thickness 0.2)
+			)
+			(justify left bottom)
+		)
+	)
 	(gr_text "Sunstang VCU 2026  Hanjing Lin   Sahil Sharma   Xiuting Shi"
-		(at 92.5 151.5 0)
+		(at 86 151 0)
 		(layer "F.SilkS")
 		(effects
@@
 		)
 	)
+	(gr_text "LV-"
+		(at 120 187 0)
+		(layer "F.SilkS")
+		(effects
+			(font
+				(size 1.25 1.25)
+				(thickness 0.2)
+			)
+			(justify left bottom)
+		)
+	)
+	(gr_text "HV-"
+		(at 127 187 0)
+		(layer "F.SilkS")
+		(effects
+			(font
+				(size 1.25 1.25)
+				(thickness 0.2)
+			)
+			(justify left bottom)
+		)
+	)
+	(gr_text "LV"
+		(at 93.5 104 0)
+		(layer "F.SilkS")
+		(effects
+			(font
+				(size 1.25 1.25)
+				(thickness 0.2)
+			)
+			(justify left bottom)
+		)
+	)
+	(gr_text "FPChrg"
+		(at 131 196 0)
+		(layer "F.SilkS")
+		(effects
+			(font
+				(size 1.25 1.25)
+				(thickness 0.2)
+			)
+			(justify left bottom)
+		)
+	)
 	(gr_text "Green LEDs\n"
 		(at 149.5 159 0)
@@
 		)
 	)
+	(gr_text "LV+"
+		(at 123.5 187 0)
+		(layer "F.SilkS")
+		(effects
+			(font
+				(size 1.25 1.25)
+				(thickness 0.2)
+			)
+			(justify left bottom)
+		)
+	)
 	(gr_text "Pre-charge\n"
 		(at 135.5 161.75 0)
@@
 		)
 	)
+	(gr_text "CM"
+		(at 120 196 0)
+		(layer "F.SilkS")
+		(effects
+			(font
+				(size 1.25 1.25)
+				(thickness 0.2)
+			)
+			(justify left bottom)
+		)
+	)
+	(gr_text "8:AccelIn  7:BrakePedalIn  6:ThermalShutoff"
+		(at 177 197 0)
+		(layer "F.SilkS")
+		(effects
+			(font
+				(size 1.25 1.25)
+				(thickness 0.2)
+			)
+			(justify left bottom)
+		)
+	)
 	(gr_text "20"
 		(at 96.5 193 0)
@@
 		)
 	)
+	(gr_text "GLEDs\n9,10\n18-20"
+		(at 164.5 193.5 0)
+		(layer "F.SilkS")
+		(effects
+			(font
+				(size 1.25 1.25)
+				(thickness 0.2)
+			)
+			(justify left bottom)
+		)
+	)
+	(gr_text "MS"
+		(at 116.5 196 0)
+		(layer "F.SilkS")
+		(effects
+			(font
+				(size 1.25 1.25)
+				(thickness 0.2)
+			)
+			(justify left bottom)
+		)
+	)
 	(gr_text "10"
 		(at 176.5 189.5 0)
@@
 		)
 	)
+	(gr_text "FAULT"
+		(at 93.5 118 0)
+		(layer "F.SilkS")
+		(effects
+			(font
+				(size 1.25 1.25)
+				(thickness 0.2)
+			)
+			(justify left bottom)
+		)
+	)
 	(gr_text "20"
 		(at 176.5 193 0)
@@
 		)
 	)
+	(gr_text "Indicator LEDs 17-20"
+		(at 91 196.5 0)
+		(layer "F.SilkS")
+		(effects
+			(font
+				(size 1.25 1.25)
+				(thickness 0.2)
+			)
+			(justify left bottom)
+		)
+	)
 	(gr_text "10"
 		(at 96.5 189.5 0)
@@
 		)
 	)
+	(gr_text "HVIL"
+		(at 93.5 113.5 0)
+		(layer "F.SilkS")
+		(effects
+			(font
+				(size 1.25 1.25)
+				(thickness 0.2)
+			)
+			(justify left bottom)
+		)
+	)
+	(gr_text "HV"
+		(at 93.5 109 0)
+		(layer "F.SilkS")
+		(effects
+			(font
+				(size 1.25 1.25)
+				(thickness 0.2)
+			)
+			(justify left bottom)
+		)
+	)
 	(gr_text "LV Switch\n"
 		(at 79.5 157.5 0)
@@
 		(layers "F.Cu" "B.Cu")
 		(free yes)
+		(tenting none)
 		(net 4)
 	)
@@
 		(drill 0.6)
 		(layers "F.Cu" "B.Cu")
+		(tenting none)
 		(net 21)
 	)
@@
 		(layers "F.Cu" "B.Cu")
 		(free yes)
+		(tenting none)
 		(net 31)
 	)
@@
 		(drill 0.6)
 		(layers "F.Cu" "B.Cu")
+		(tenting none)
 		(net 130)
 	)
